Commit message: Add ros2_control

File: mobro_description/urdf/gazebo_depth_camera.xacro (robot description, xacro)
@@ -6,9 +6,4 @@
       <origin rpy="0 0 0" xyz="0 0 0"/>
     </xacro:inertial_box>
-    <!-- <inertial>
-      <mass value="0.1"/>
-      <origin rpy="0 0 0" xyz="0 0 0"/>
-      <inertia ixx="0.0003866666666666667" ixy="0" ixz="0" iyy="0.00010666666666666668" iyz="0" izz="0.0003866666666666667"/>
-    </inertial> -->
     <visual>
       <origin rpy="0 0 0" xyz="0 0 0"/>
@@ -35,9 +30,6 @@
     <parent link="camera"/>
     <child link="camera_optical"/>
-    <!-- Rotate to align with ROS optical frame convention:
-           X: Right, Y: Down, Z: Forward -->
     <origin rpy="-1.5707963267948966 0 -1.5707963267948966" xyz="0 0 0"/>
   </joint>
-  <!-- Gazebo Camera Plugin -->
   <gazebo reference="camera">
     <material>Gazebo/Blue</material>

File: mobro_description/urdf/gazebo_lidar_rgbd.xacro (robot description, xacro)
@@ -24,5 +24,4 @@
     <origin rpy="0 0 0" xyz="-0.1 0 0.22"/>
   </joint>
-  <!-- Gazebo Lidar Plugin -->
   <gazebo reference="lidar">
     <material>Gazebo/Red</material>
@@ -75,9 +74,4 @@
       <origin rpy="0 0 0" xyz="0 0 0"/>
     </xacro:inertial_box>
-    <!-- <inertial>
-      <mass value="0.1"/>
-      <origin rpy="0 0 0" xyz="0 0 0"/>
-      <inertia ixx="0.0003866666666666667" ixy="0" ixz="0" iyy="0.00010666666666666668" iyz="0" izz="0.0003866666666666667"/>
-    </inertial> -->
     <visual>
       <origin rpy="0 0 0" xyz="0 0 0"/>
@@ -104,9 +98,6 @@
     <parent link="camera"/>
     <child link="camera_optical"/>
-    <!-- Rotate to align with ROS optical frame convention:
-           X: Right, Y: Down, Z: Forward -->
     <origin rpy="-1.5707963267948966 0 -1.5707963267948966" xyz="0 0 0"/>
   </joint>
-  <!-- Gazebo Camera Plugin -->
   <gazebo reference="camera">
     <material>Gazebo/Blue</material>

File: mobro_description/urdf/gazebo_rgb_camera.xacro (robot description, xacro)
@@ -6,9 +6,4 @@
       <origin rpy="0 0 0" xyz="0 0 0"/>
     </xacro:inertial_box>
-    <!-- <inertial>
-      <mass value="0.1"/>
-      <origin rpy="0 0 0" xyz="0 0 0"/>
-      <inertia ixx="0.0003866666666666667" ixy="0" ixz="0" iyy="0.00010666666666666668" iyz="0" izz="0.0003866666666666667"/>
-    </inertial> -->
     <visual>
       <origin rpy="0 0 0" xyz="0 0 0"/>
@@ -35,6 +30,4 @@
     <parent link="camera"/>
     <child link="camera_optical"/>
-    <!-- Rotate to align with ROS optical frame convention:
-           X: Right, Y: Down, Z: Forward -->
     <origin rpy="-1.5707963267948966 0 -1.5707963267948966" xyz="0 0 0"/>
   </joint>

File: mobro_description/urdf/inertial_macro.xacro (robot description, xacro)
@@ -1,4 +1,4 @@
 <?xml version="1.0"?>
-<robot xmlns:xacro="http://www.ros.org/wiki/xacro" >
+<robot xmlns:xacro="http://www.ros.org/wiki/xacro">
     <!-- Inertial calculations in https://en.wikipedia.org/wiki/List_of_moments_of_inertia -->
     <!-- These make use of xacro's mathematical functionality -->

File: mobro_description/urdf/mobro_core.xacro (robot description, xacro)
@@ -1,5 +1,5 @@
 <?xml version="1.0" ?>
 <robot xmlns:xacro="http://www.ros.org/wiki/xacro" name="mobro">
-  <xacro:include filename="$(find mobro_description)/urdf/inertial_macro.xacro" />
+  <xacro:include filename="$(find mobro_description)/urdf/inertial_macro.xacro"/>
   <material name="Gray">
     <color rgba="0.5 0.5 0.5 1.0"/>
@@ -47,6 +47,4 @@
   <gazebo reference="base_link">
       <material>Gazebo/White</material>
-      <!-- <mu1>0.5</mu1>
-      <mu2>0.5</mu2> -->
   </gazebo>
   <joint name="left_joint" type="continuous">

File: mobro_description/urdf/robot.urdf.xacro (robot description, xacro)
@@ -2,6 +2,6 @@
 <robot xmlns:xacro="http://www.ros.org/wiki/xacro" name="mobro">
   <xacro:include filename="$(find mobro_description)/urdf/mobro_core.xacro"/>
-  <xacro:include filename="$(find mobro_description)/urdf/gazebo_control.xacro"/>
   <xacro:include filename="$(find mobro_description)/urdf/gazebo_lidar_rgbd.xacro"/>
+  <xacro:include filename="$(find mobro_description)/urdf/ros2_control.xacro"/>
   <!-- <xacro:include filename="$(find mobro_description)/urdf/gazebo_rgb_camera.xacro"/> -->
   <!-- <xacro:include filename="$(find mobro_description)/urdf/gazebo_depth_camera.xacro"/> -->
