Commit message: Resize the robot and update README

File: mobro_description/urdf/gazebo_2D_lidar.xacro (robot description, xacro)
@@ -1,14 +1,12 @@
 <?xml version="1.0"?>
 <robot xmlns:xacro="http://www.ros.org/wiki/xacro">
-<link name="lidar">
-    <inertial>
-      <mass value="0.2"/>
+  <link name="lidar">
+    <xacro:inertial_cylinder mass="0.2" length="0.04" radius="0.04">
       <origin rpy="0 0 0" xyz="0 0 0"/>
-      <inertia ixx="0.0006066666666666668" ixy="0" ixz="0" iyy="0.0006066666666666668" iyz="0" izz="0.0010000000000000002"/>
-    </inertial>
+    </xacro:inertial_cylinder>
     <visual>
       <origin rpy="0 0 0" xyz="0 0 0"/>
       <geometry>
-        <cylinder length="0.08" radius="0.1"/>
+        <cylinder length="0.04" radius="0.04"/>
       </geometry>
       <material name="Red"/>
@@ -17,15 +15,16 @@
       <origin rpy="0 0 0" xyz="0 0 0"/>
       <geometry>
-        <cylinder length="0.08" radius="0.1"/>
+        <cylinder length="0.04" radius="0.04"/>
       </geometry>
     </collision>
   </link>
   <joint name="lidar_joint" type="fixed">
-    <parent link="chassis"/>
+    <parent link="base_link"/>
     <child link="lidar"/>
-    <origin rpy="0 0 0" xyz="0.6 0 0.3"/>
+    <origin rpy="0 0 0" xyz="-0.1 0 0.22"/>
   </joint>
   <!-- Gazebo Lidar Plugin -->
-    <gazebo reference="lidar">
+  <gazebo reference="lidar">
+    <material>Gazebo/Red</material>
     <sensor type="ray" name="lidar_sensor">
       <pose>0 0 0 0 0 0</pose>
@@ -36,19 +35,13 @@
           <horizontal>
             <samples>360</samples>
-            <resolution>1</resolution>
+            <resolution>1.000000</resolution>
             <min_angle>-3.1415</min_angle>
             <max_angle>3.1415</max_angle>
           </horizontal>
-          <!-- <vertical>
-            <samples>10</samples>
-              <resolution>1</resolution>
-              <min_angle>0</min_angle>
-              <max_angle>3*PI/180.0</max_angle>
-          </vertical> -->
         </scan>
         <range>
-          <min>0.3</min>
+          <min>0.05</min>
           <max>10.0</max>
-          <resolution>0.01</resolution>
+          <!-- <resolution>0.01</resolution> -->
         </range>
         <noise>
@@ -56,14 +49,11 @@
           <mean>0.0</mean>
           <stddev>0.01</stddev>
-      </noise>
+        </noise>
       </ray>
       <plugin name="lidar_plugin" filename="libgazebo_ros_ray_sensor.so">
         <ros>
-          <namespace>/</namespace>
+          <!-- <namespace>/</namespace> -->
           <remapping>~/out:=scan</remapping>
-          <!-- <remapping>~/out:=pointcloud2</remapping> -->
         </ros>
-        <!-- <output_type>sensor_msgs/PointCloud2</output_type>
-        <min_intensity>100.0</min_intensity> -->
         <output_type>sensor_msgs/LaserScan</output_type>
         <frame_name>lidar</frame_name>
@@ -71,6 +61,3 @@
     </sensor>
   </gazebo>
-  <gazebo reference="lidar">
-      <material>Gazebo/Red</material>
-  </gazebo>
 </robot>

File: mobro_description/urdf/gazebo_3D_lidar.xacro (robot description, xacro)
@@ -1,14 +1,12 @@
 <?xml version="1.0"?>
 <robot xmlns:xacro="http://www.ros.org/wiki/xacro">
-<link name="lidar">
-    <inertial>
-      <mass value="0.2"/>
+  <link name="lidar">
+    <xacro:inertial_cylinder mass="0.2" length="0.04" radius="0.04">
       <origin rpy="0 0 0" xyz="0 0 0"/>
-      <inertia ixx="0.0006066666666666668" ixy="0" ixz="0" iyy="0.0006066666666666668" iyz="0" izz="0.0010000000000000002"/>
-    </inertial>
+    </xacro:inertial_cylinder>
     <visual>
       <origin rpy="0 0 0" xyz="0 0 0"/>
       <geometry>
-        <cylinder length="0.08" radius="0.1"/>
+        <cylinder length="0.04" radius="0.04"/>
       </geometry>
       <material name="Red"/>
@@ -17,15 +15,16 @@
       <origin rpy="0 0 0" xyz="0 0 0"/>
       <geometry>
-        <cylinder length="0.08" radius="0.1"/>
+        <cylinder length="0.04" radius="0.04"/>
       </geometry>
     </collision>
   </link>
   <joint name="lidar_joint" type="fixed">
-    <parent link="chassis"/>
+    <parent link="base_link"/>
     <child link="lidar"/>
-    <origin rpy="0 0 0" xyz="0.6 0 0.3"/>
+    <origin rpy="0 0 0" xyz="-0.1 0 0.22"/>
   </joint>
   <!-- Gazebo Lidar Plugin -->
-    <gazebo reference="lidar">
+  <gazebo reference="lidar">
+    <material>Gazebo/Red</material>
     <sensor type="ray" name="lidar_sensor">
       <pose>0 0 0 0 0 0</pose>
@@ -36,5 +35,5 @@
           <horizontal>
             <samples>360</samples>
-            <resolution>1</resolution>
+            <!-- <resolution>1</resolution> -->
             <min_angle>-3.1415</min_angle>
             <max_angle>3.1415</max_angle>
@@ -42,23 +41,23 @@
           <vertical>
             <samples>10</samples>
-              <resolution>1</resolution>
-              <min_angle>0</min_angle>
-              <max_angle>3*PI/180.0</max_angle>
+              <!-- <resolution>1</resolution> -->
+            <min_angle>0</min_angle>
+            <max_angle>3*PI/180.0</max_angle>
           </vertical>
         </scan>
         <range>
-          <min>0.3</min>
+          <min>0.05</min>
           <max>10.0</max>
-          <resolution>0.01</resolution>
+          <!-- <resolution>0.01</resolution> -->
         </range>
-        <noise>
+        <!-- <noise>
           <type>gaussian</type>
           <mean>0.0</mean>
           <stddev>0.01</stddev>
-      </noise>
+        </noise> -->
       </ray>
       <plugin name="lidar_plugin" filename="libgazebo_ros_ray_sensor.so">
         <ros>
-          <namespace>/</namespace>
+          <!-- <namespace>/</namespace> -->
           <!-- <remapping>~/out:=scan</remapping> -->
           <remapping>~/out:=pointcloud2</remapping>
@@ -71,6 +70,3 @@
     </sensor>
   </gazebo>
-  <gazebo reference="lidar">
-      <material>Gazebo/Red</material>
-  </gazebo>
 </robot>

File: mobro_description/urdf/gazebo_control.xacro (robot description, xacro)
@@ -1,5 +1,5 @@
 <?xml version="1.0"?>
 <robot xmlns:xacro="http://www.ros.org/wiki/xacro">
-    <gazebo>
+  <gazebo>
     <plugin name="differential_drive_controller" filename="libgazebo_ros_diff_drive.so">
       <ros>
@@ -10,19 +10,18 @@
       <left_joint>left_joint</left_joint>
       <right_joint>right_joint</right_joint>
-      <odometry_frame>odom</odometry_frame>
       <!-- Limits -->
-      <max_wheel_torque>20</max_wheel_torque>
+      <max_wheel_torque>200</max_wheel_torque>
       <max_wheel_acceleration>1.0</max_wheel_acceleration>
-      <wheel_separation>0.92</wheel_separation>
-      <wheel_diameter>0.44</wheel_diameter>
+      <wheel_separation>0.44</wheel_separation>
+      <wheel_diameter>0.1</wheel_diameter>
       <!-- Output -->
-      <robot_base_frame>base_link</robot_base_frame>
+      <robot_base_frame>base_footprint</robot_base_frame>
       <odometry_frame>odom</odometry_frame>
       <publish_odom>true</publish_odom>
       <publish_odom_tf>true</publish_odom_tf>
-      <publish_wheel_tf>true</publish_wheel_tf>
+      <publish_wheel_tf>false</publish_wheel_tf>
     </plugin>
   </gazebo>
-  <gazebo>
+  <!-- <gazebo>
     <plugin name="joint_states" filename="libgazebo_ros_joint_state_publisher.so">
       <ros>
@@ -32,6 +31,5 @@
       <joint_name>right_joint</joint_name>
       <joint_name>left_joint</joint_name>
-      <!-- <joint_name>front_caster_joint</joint_name> -->
     </plugin>
-  </gazebo>
+  </gazebo> -->
 </robot>

File: mobro_description/urdf/gazebo_depth_camera.xacro (robot description, xacro)
@@ -3,13 +3,16 @@
   <!-- Camera Frame -->
   <link name="camera">
-    <inertial>
+    <xacro:inertial_box mass="0.1" x="0.03" y="0.1" z="0.03">
+      <origin rpy="0 0 0" xyz="0 0 0"/>
+    </xacro:inertial_box>
+    <!-- <inertial>
       <mass value="0.1"/>
       <origin rpy="0 0 0" xyz="0 0 0"/>
       <inertia ixx="0.0003866666666666667" ixy="0" ixz="0" iyy="0.00010666666666666668" iyz="0" izz="0.0003866666666666667"/>
-    </inertial>
+    </inertial> -->
     <visual>
       <origin rpy="0 0 0" xyz="0 0 0"/>
       <geometry>
-        <box size="0.08 0.2 0.08"/>
+        <box size="0.03 0.1 0.03"/>
       </geometry>
       <material name="Blue"/>
@@ -18,12 +21,12 @@
       <origin rpy="0 0 0" xyz="0 0 0"/>
       <geometry>
-        <box size="0.08 0.2 0.08"/>
+        <box size="0.03 0.1 0.03"/>
       </geometry>
     </collision>
   </link>
   <joint name="camera_joint" type="fixed">
-    <parent link="chassis"/>
+    <parent link="base_link"/>
     <child link="camera"/>
-    <origin rpy="0 0 0" xyz="1.2 0 0.15"/>
+    <origin rpy="0 0 0" xyz="0.115 0 0.1"/>
   </joint>
   <!-- Camera Optical Frame -->
@@ -38,4 +41,5 @@
   <!-- Gazebo Camera Plugin -->
   <gazebo reference="camera">
+    <material>Gazebo/Blue</material>
     <sensor name="camera" type="depth">
       <pose> 0 0 0 0 0 0 </pose>
@@ -61,6 +65,3 @@
     </sensor>
   </gazebo>
-  <gazebo reference="camera">
-      <material>Gazebo/Blue</material>
-  </gazebo>
 </robot>

File: mobro_description/urdf/gazebo_lidar_rgbd.xacro (robot description, xacro)
@@ -1,14 +1,12 @@
 <?xml version="1.0"?>
 <robot xmlns:xacro="http://www.ros.org/wiki/xacro">
-<link name="lidar">
-    <inertial>
-      <mass value="0.2"/>
+  <link name="lidar">
+    <xacro:inertial_cylinder mass="0.2" length="0.04" radius="0.04">
       <origin rpy="0 0 0" xyz="0 0 0"/>
-      <inertia ixx="0.0006066666666666668" ixy="0" ixz="0" iyy="0.0006066666666666668" iyz="0" izz="0.0010000000000000002"/>
-    </inertial>
+    </xacro:inertial_cylinder>
     <visual>
       <origin rpy="0 0 0" xyz="0 0 0"/>
       <geometry>
-        <cylinder length="0.08" radius="0.1"/>
+        <cylinder length="0.04" radius="0.04"/>
       </geometry>
       <material name="Red"/>
@@ -17,15 +15,16 @@
       <origin rpy="0 0 0" xyz="0 0 0"/>
       <geometry>
-        <cylinder length="0.08" radius="0.1"/>
+        <cylinder length="0.04" radius="0.04"/>
       </geometry>
     </collision>
   </link>
   <joint name="lidar_joint" type="fixed">
-    <parent link="chassis"/>
+    <parent link="base_link"/>
     <child link="lidar"/>
-    <origin rpy="0 0 0" xyz="0.6 0 0.3"/>
+    <origin rpy="0 0 0" xyz="-0.1 0 0.22"/>
   </joint>
   <!-- Gazebo Lidar Plugin -->
-    <gazebo reference="lidar">
+  <gazebo reference="lidar">
+    <material>Gazebo/Red</material>
     <sensor type="ray" name="lidar_sensor">
       <pose>0 0 0 0 0 0</pose>
@@ -36,5 +35,5 @@
           <horizontal>
             <samples>360</samples>
-            <resolution>1</resolution>
+            <resolution>1.000000</resolution>
             <min_angle>-3.1415</min_angle>
             <max_angle>3.1415</max_angle>
@@ -48,7 +47,7 @@
         </scan>
         <range>
-          <min>0.3</min>
+          <min>0.05</min>
           <max>10.0</max>
-          <resolution>0.01</resolution>
+          <!-- <resolution>0.01</resolution> -->
         </range>
         <noise>
@@ -56,9 +55,9 @@
           <mean>0.0</mean>
           <stddev>0.01</stddev>
-      </noise>
+        </noise>
       </ray>
       <plugin name="lidar_plugin" filename="libgazebo_ros_ray_sensor.so">
         <ros>
-          <namespace>/</namespace>
+          <!-- <namespace>/</namespace> -->
           <remapping>~/out:=scan</remapping>
           <!-- <remapping>~/out:=pointcloud2</remapping> -->
@@ -71,18 +70,18 @@
     </sensor>
   </gazebo>
-  <gazebo reference="lidar">
-      <material>Gazebo/Red</material>
-  </gazebo>
   <!-- Camera Frame -->
   <link name="camera">
-    <inertial>
+    <xacro:inertial_box mass="0.1" x="0.03" y="0.1" z="0.03">
+      <origin rpy="0 0 0" xyz="0 0 0"/>
+    </xacro:inertial_box>
+    <!-- <inertial>
       <mass value="0.1"/>
       <origin rpy="0 0 0" xyz="0 0 0"/>
       <inertia ixx="0.0003866666666666667" ixy="0" ixz="0" iyy="0.00010666666666666668" iyz="0" izz="0.0003866666666666667"/>
-    </inertial>
+    </inertial> -->
     <visual>
       <origin rpy="0 0 0" xyz="0 0 0"/>
       <geometry>
-        <box size="0.08 0.2 0.08"/>
+        <box size="0.03 0.1 0.03"/>
       </geometry>
       <material name="Blue"/>
@@ -91,12 +90,12 @@
       <origin rpy="0 0 0" xyz="0 0 0"/>
       <geometry>
-        <box size="0.08 0.2 0.08"/>
+        <box size="0.03 0.1 0.03"/>
       </geometry>
     </collision>
   </link>
   <joint name="camera_joint" type="fixed">
-    <parent link="chassis"/>
+    <parent link="base_link"/>
     <child link="camera"/>
-    <origin rpy="0 0 0" xyz="1.2 0 0.15"/>
+    <origin rpy="0 0 0" xyz="0.115 0 0.1"/>
   </joint>
   <!-- Camera Optical Frame -->
@@ -111,4 +110,5 @@
   <!-- Gazebo Camera Plugin -->
   <gazebo reference="camera">
+    <material>Gazebo/Blue</material>
     <sensor name="camera" type="depth">
       <pose> 0 0 0 0 0 0 </pose>
@@ -134,6 +134,3 @@
     </sensor>
   </gazebo>
-  <gazebo reference="camera">
-      <material>Gazebo/Blue</material>
-  </gazebo>
 </robot>

File: mobro_description/urdf/gazebo_rgb_camera.xacro (robot description, xacro)
@@ -3,13 +3,16 @@
   <!-- Camera Frame -->
   <link name="camera">
-    <inertial>
+    <xacro:inertial_box mass="0.1" x="0.03" y="0.1" z="0.03">
+      <origin rpy="0 0 0" xyz="0 0 0"/>
+    </xacro:inertial_box>
+    <!-- <inertial>
       <mass value="0.1"/>
       <origin rpy="0 0 0" xyz="0 0 0"/>
       <inertia ixx="0.0003866666666666667" ixy="0" ixz="0" iyy="0.00010666666666666668" iyz="0" izz="0.0003866666666666667"/>
-    </inertial>
+    </inertial> -->
     <visual>
       <origin rpy="0 0 0" xyz="0 0 0"/>
       <geometry>
-        <box size="0.08 0.2 0.08"/>
+        <box size="0.03 0.1 0.03"/>
       </geometry>
       <material name="Blue"/>
@@ -18,12 +21,12 @@
       <origin rpy="0 0 0" xyz="0 0 0"/>
       <geometry>
-        <box size="0.08 0.2 0.08"/>
+        <box size="0.03 0.1 0.03"/>
       </geometry>
     </collision>
   </link>
   <joint name="camera_joint" type="fixed">
-    <parent link="chassis"/>
+    <parent link="base_link"/>
     <child link="camera"/>
-    <origin rpy="0 0 0" xyz="1.2 0 0.15"/>
+    <origin rpy="0 0 0" xyz="0.115 0 0.1"/>
   </joint>
   <!-- Camera Optical Frame -->
@@ -37,4 +40,5 @@
   </joint>
   <gazebo reference="camera">
+    <material>Gazebo/Blue</material>
     <sensor type="camera" name="camera_sensor">
       <pose>0 0 0 0 0 0</pose>

File: mobro_description/urdf/mobro_core.xacro (robot description, xacro)
@@ -20,43 +20,30 @@
     <color rgba="1.0 1.0 1.0 1.0"/>
   </material>
-  <!-- <gazebo reference="lidar">
-      <material>Gazebo/Red</material>
-  </gazebo>
-  <gazebo reference="camera">
-      <material>Gazebo/Blue</material>
-  </gazebo> -->
-  <link name="base_link">
+  <link name="base_footprint">
   </link>
   <joint name="base_footprint_joint" type="fixed">
-    <parent link="base_link"/>
-    <child link="base_footprint"/>
+    <parent link="base_footprint"/>
+    <child link="base_link"/>
     <origin xyz="0 0 0" rpy="0 0 0"/>
   </joint>
-  <link name="base_footprint">
-  </link>
-  <joint name="base_to_chassis" type="fixed">
-    <parent link="base_link"/>
-    <child link="chassis"/>
-    <origin rpy="0 0 0" xyz="-0.9 0 0"/>
-  </joint>
-  <link name="chassis">
-    <xacro:inertial_box mass="1.0" x="1.2" y="0.8" z="0.3">
-      <origin rpy="0 0 0" xyz="0.6 0 0.1"/>
+  <link name="base_link">
+    <xacro:inertial_box mass="1.0" x="0.4" y="0.4" z="0.2">
+      <origin rpy="0 0 0" xyz="-0.1 0 0.1"/>
     </xacro:inertial_box>
     <visual>
-      <origin rpy="0 0 0" xyz="0.6 0 0.1"/>
+      <origin rpy="0 0 0" xyz="-0.1 0 0.1"/>
       <geometry>
-        <box size="1.2 0.8 0.3"/>
+        <box size="0.4 0.4 0.2"/>
       </geometry>
       <material name="Gray"/>
     </visual>
     <collision>
-      <origin rpy="0 0 0" xyz="0.6 0 0.1"/>
+      <origin rpy="0 0 0" xyz="-0.1 0 0.1"/>
       <geometry>
-        <box size="1.2 0.8 0.3"/>
+        <box size="0.4 0.4 0.2"/>
       </geometry>
     </collision>
   </link>
-  <gazebo reference="chassis">
+  <gazebo reference="base_link">
       <material>Gazebo/White</material>
       <!-- <mu1>0.5</mu1>
@@ -66,9 +53,9 @@
     <parent link="base_link"/>
     <child link="left_wheel"/>
-    <origin rpy="-${pi/2} 0 0" xyz="0 0.46 0"/>
+    <origin rpy="-${pi/2} 0 0" xyz="0 0.22 0"/>
     <axis xyz="0 0 1"/>
   </joint>
   <link name="left_wheel">
-    <xacro:inertial_cylinder mass="0.5" length="0.12" radius="0.22">
+    <xacro:inertial_cylinder mass="0.5" length="0.04" radius="0.05">
       <origin rpy="0 0 0" xyz="0 0 0"/>
     </xacro:inertial_cylinder>
@@ -76,5 +63,5 @@
       <origin rpy="0 0 0" xyz="0 0 0"/>
       <geometry>
-        <cylinder length="0.12" radius="0.22"/>
+        <cylinder length="0.04" radius="0.05"/>
       </geometry>
       <material name="Black"/>
@@ -83,5 +70,5 @@
       <origin rpy="0 0 0" xyz="0 0 0"/>
       <geometry>
-        <cylinder length="0.12" radius="0.22"/>
+        <cylinder length="0.04" radius="0.05"/>
       </geometry>
     </collision>
@@ -95,9 +82,9 @@
     <parent link="base_link"/>
     <child link="right_wheel"/>
-    <origin rpy="${pi/2} 0 0" xyz="0 -0.46 0"/>
+    <origin rpy="${pi/2} 0 0" xyz="0 -0.22 0"/>
     <axis xyz="0 0 -1"/>
   </joint>
   <link name="right_wheel">
-    <xacro:inertial_cylinder mass="0.5" length="0.12" radius="0.22">
+    <xacro:inertial_cylinder mass="0.5" length="0.04" radius="0.05">
       <origin rpy="0 0 0" xyz="0 0 0"/>
     </xacro:inertial_cylinder>
@@ -105,5 +92,5 @@
       <origin rpy="0 0 0" xyz="0 0 0"/>
       <geometry>
-        <cylinder length="0.12" radius="0.22"/>
+        <cylinder length="0.04" radius="0.05"/>
       </geometry>
       <material name="Black"/>
@@ -112,5 +99,5 @@
       <origin rpy="0 0 0" xyz="0 0 0"/>
       <geometry>
-        <cylinder length="0.12" radius="0.22"/>
+        <cylinder length="0.04" radius="0.05"/>
       </geometry>
     </collision>
@@ -122,10 +109,10 @@
   </gazebo>
   <joint name="front_caster_joint" type="fixed">
-    <parent link="chassis"/>
+    <parent link="base_link"/>
     <child link="front_caster_wheel"/>
-    <origin rpy="0 0 0" xyz="0.15 0 -0.11"/>
+    <origin rpy="0 0 0" xyz="-0.225 0 0"/>
   </joint>
   <link name="front_caster_wheel">
-    <xacro:inertial_sphere mass="0.3" radius="0.11">
+    <xacro:inertial_sphere mass="0.5" radius="0.05">
       <origin rpy="0 0 0" xyz="0 0 0"/>
     </xacro:inertial_sphere>
@@ -133,5 +120,5 @@
       <origin rpy="0 0 0" xyz="0 0 0"/>
       <geometry>
-        <sphere radius="0.11"/>
+        <sphere radius="0.05"/>
       </geometry>
       <material name="Black"/>
@@ -140,5 +127,5 @@
       <origin rpy="0 0 0" xyz="0 0 0"/>
       <geometry>
-        <sphere radius="0.11"/>
+        <sphere radius="0.05"/>
       </geometry>
     </collision>

File: mobro_description/urdf/robot.urdf.xacro (robot description, xacro)
@@ -3,8 +3,8 @@
   <xacro:include filename="$(find mobro_description)/urdf/mobro_core.xacro"/>
   <xacro:include filename="$(find mobro_description)/urdf/gazebo_control.xacro"/>
-  <!-- <xacro:include filename="$(find mobro_description)/urdf/gazebo_lidar_rgbd.xacro"/> -->
-  <xacro:include filename="$(find mobro_description)/urdf/gazebo_rgb_camera.xacro"/>
+  <xacro:include filename="$(find mobro_description)/urdf/gazebo_lidar_rgbd.xacro"/>
+  <!-- <xacro:include filename="$(find mobro_description)/urdf/gazebo_rgb_camera.xacro"/> -->
   <!-- <xacro:include filename="$(find mobro_description)/urdf/gazebo_depth_camera.xacro"/> -->
-  <xacro:include filename="$(find mobro_description)/urdf/gazebo_2D_lidar.xacro"/>
+  <!-- <xacro:include filename="$(find mobro_description)/urdf/gazebo_2D_lidar.xacro"/> -->
   <!-- <xacro:include filename="$(find mobro_description)/urdf/gazebo_3D_lidar.xacro"/> -->
 </robot>
