Commit message: Update README and add the gazebo parameter

File: mobro_description/urdf/gazebo_2D_lidar.xacro (robot description, xacro)
@@ -29,5 +29,5 @@
     <sensor type="ray" name="lidar_sensor">
       <pose>0 0 0 0 0 0</pose>
-      <visualize>true</visualize>
+      <visualize>false</visualize>
       <update_rate>10</update_rate>
       <ray>

File: mobro_description/urdf/mobro_core.xacro (robot description, xacro)
@@ -65,8 +65,15 @@
       <material name="Black"/>
     </visual>
+    <!-- <collision>
+      <origin rpy="0 0 0" xyz="0 0 0"/>
+      <geometry>
+        <cylinder length="0.04" radius="0.05"/>
+      </geometry>
+    </collision> -->
+    <!-- set sphere since it is simulation which has ideal conditions -->
     <collision>
       <origin rpy="0 0 0" xyz="0 0 0"/>
       <geometry>
-        <cylinder length="0.04" radius="0.05"/>
+        <sphere radius="0.05"/>
       </geometry>
     </collision>
@@ -74,6 +81,6 @@
   <gazebo reference="left_wheel">
       <material>Gazebo/Black</material>
-      <mu1>0.5</mu1>
-      <mu2>0.5</mu2>
+      <mu1>1.0</mu1>
+      <mu2>1.0</mu2>
   </gazebo>
   <joint name="right_joint" type="continuous">
@@ -94,8 +101,15 @@
       <material name="Black"/>
     </visual>
+    <!-- <collision>
+      <origin rpy="0 0 0" xyz="0 0 0"/>
+      <geometry>
+        <cylinder length="0.04" radius="0.05"/>
+      </geometry>
+    </collision> -->
+    <!-- set sphere since it is simulation which has ideal conditions -->
     <collision>
       <origin rpy="0 0 0" xyz="0 0 0"/>
       <geometry>
-        <cylinder length="0.04" radius="0.05"/>
+        <sphere radius="0.05"/>
       </geometry>
     </collision>
@@ -103,6 +117,6 @@
   <gazebo reference="right_wheel">
       <material>Gazebo/Black</material>
-      <mu1>0.5</mu1>
-      <mu2>0.5</mu2>
+      <mu1>1.0</mu1>
+      <mu2>1.0</mu2>
   </gazebo>
   <joint name="front_caster_joint" type="fixed">
@@ -131,6 +145,6 @@
   <gazebo reference="front_caster_wheel">
       <material>Gazebo/Black</material>
-      <mu1>0.2</mu1>
-      <mu2>0.2</mu2>
+      <mu1>0.001</mu1>
+      <mu2>0.001</mu2>
   </gazebo>
 </robot>

File: mobro_description/urdf/robot.urdf.xacro (robot description, xacro)
@@ -1,10 +1,18 @@
 <?xml version="1.0" ?>
 <robot xmlns:xacro="http://www.ros.org/wiki/xacro" name="mobro">
+  <!-- robot base -->
   <xacro:include filename="$(find mobro_description)/urdf/mobro_core.xacro"/>
-  <xacro:include filename="$(find mobro_description)/urdf/gazebo_lidar_rgbd.xacro"/>
-  <xacro:include filename="$(find mobro_description)/urdf/ros2_control.xacro"/>
-  <!-- <xacro:include filename="$(find mobro_description)/urdf/gazebo_rgb_camera.xacro"/> -->
+  <!-- gazebo plugins -->
+  <xacro:if value="$(arg use_ros2_control)">
+    <xacro:include filename="$(find mobro_description)/urdf/ros2_control.xacro"/>
+  </xacro:if>
+  <xacro:unless value="$(arg use_ros2_control)">
+    <xacro:include filename="$(find mobro_description)/urdf/gazebo_control.xacro"/>
+  </xacro:unless>
+  <!-- sensor plugins -->
+  <!-- <xacro:include filename="$(find mobro_description)/urdf/gazebo_lidar_rgbd.xacro"/> -->
+  <xacro:include filename="$(find mobro_description)/urdf/gazebo_rgb_camera.xacro"/>
   <!-- <xacro:include filename="$(find mobro_description)/urdf/gazebo_depth_camera.xacro"/> -->
-  <!-- <xacro:include filename="$(find mobro_description)/urdf/gazebo_2D_lidar.xacro"/> -->
+  <xacro:include filename="$(find mobro_description)/urdf/gazebo_2D_lidar.xacro"/>
   <!-- <xacro:include filename="$(find mobro_description)/urdf/gazebo_3D_lidar.xacro"/> -->
 </robot>
